File: Starbie/Starbie.kicad_pcb (KiCad board)
At the start: 2 copper layers, 114.5 x 104 mm, 7 parts, among them J1 Conn_01x04_Pin, J2 Conn_01x08_Pin, SW1 SW_Push, SW2 SW_Push, U1 XIAO-ESP32-C3-SMD, U2 DHT11

Commit message: re routed and added art
Parts:
- added G***: LOGO, LOGO, F.Cu at (101.0, 119.5)
- added G***: LOGO, LOGO, F.Cu at (110.0, 86.5)
- added G***: LOGO, LOGO, F.Cu at (145.5, 141.5)
- moved SW2 15.9 mm to (100.1, 130.9)
- moved J1 13.7 mm to (120.3, 89.0)
- moved R1 10.0 mm to (114.2, 72.0)
- moved SW1 9.74 mm to (90.1, 97.8)
- moved U1 9.50 mm to (129.9, 128.5)
- moved U2 8.06 mm to (152.0, 106.5)
- moved J2 7.94 mm to (142.5, 95.8)
Routing:
- net /SCL: track 117.0 -> 300.1 mm
- net GND: track 283.6 -> 159.4 mm
- net /SDA: track 127.1 -> 52.5 mm
- net +3.3V: track 222.1 -> 192.5 mm
- net /GPIO3: track 23.9 -> 45.2 mm
- net /DHT11 DATA: track 71.7 -> 87.0 mm
- net /GPI02: track 43.2 -> 52.8 mm
Other:
- board size 114.5 x 104 mm -> 114.5 x 102 mm

Commit message: added usbc keyboard support
(kinda)
Parts:
- removed the G*** at (101.0, 119.5)
- removed the G*** at (110.0, 86.5)
- added J3: USB_C_Receptacle_USB2.0_14P, Connector_USB:USB_C_Receptacle_HRO_TYPE-C-31-M-17, F.Cu at (119.0, 157.0)
- added R2: 5k, Package_DIP:DIP-8_W7.62mm, F.Cu at (141.7, 159.2)
- added R3: 5k, Package_DIP:DIP-8_W7.62mm, F.Cu at (87.2, 160.2)
Connections:
- U1 pad 8: unconnected-(U1-D7-Pad8) -> /pair2
- U1 pad 9: unconnected-(U1-D8-Pad9) -> /pair1
Routing:
- net GND: track 159.4 -> 309.3 mm
- net +5V: track 0.00 -> 54.3 mm
- net /ng: track 0.00 -> 35.0 mm
- net /groundi: track 0.00 -> 24.0 mm
Other:
- board size 114.5 x 102 mm -> 132.5 x 127.5 mm

Commit message: added more and changed shape
Parts:
- moved G*** 84.5 mm to (146.0, 57.0)
- moved R2 42.1 mm to (156.2, 119.7)
- moved SW2 38.4 mm to (77.5, 99.9)
- moved SW1 28.3 mm to (77.3, 72.5)
- moved R3 22.4 mm to (84.5, 138.0)
- moved U2 19.5 mm to (159.5, 88.5)
- moved J2 17.3 mm to (142.3, 78.4)
- moved U1 15.9 mm to (114.0, 130.0)
- moved J1 8.59 mm to (113.0, 84.5)
- moved R1 5.52 mm to (110.4, 68.0)
- moved J3 4.18 mm to (122.8, 155.3)
Routing:
- net /SCL: track 300.1 -> 68.2 mm
- net GND: track 309.3 -> 438.6 mm
- net /GPI02: track 52.8 -> 137.3 mm
- net /DHT11 DATA: track 87.0 -> 141.5 mm
- net /groundi: track 24.0 -> 71.4 mm
- net /ng: track 35.0 -> 74.1 mm
- net +3.3V: track 192.5 -> 153.9 mm
- net +5V: track 54.3 -> 25.7 mm
- net /SDA: track 52.5 -> 68.3 mm
- net /GPIO3: track 45.2 -> 46.8 mm
- net (no net): track 0.00 -> 1.40 mm
Other:
- board size 132.5 x 127.5 mm -> 140 x 145.5 mm

Commit message: added a lot
Parts:
- added :3: LOGO, Imported Parts:abcd, F.Cu at (150.7, 109.9)
- added :3: LOGO, Imported Parts:abcd, F.Cu at (163.4, 71.7)
- added :3: LOGO, Imported Parts:abcd, F.Cu at (147.0, 110.5)
- added :3: LOGO, Imported Parts:abcd, F.Cu at (167.6, 72.9)
- added :3c: LOGO, Imported Parts:def, F.Cu at (84.5, 129.5)
- added :3c: LOGO, Imported Parts:def, F.Cu at (147.0, 138.0)
- moved U1 25.5 mm to (103.0, 153.0), turned to -135 degrees
- moved J3 10.3 mm to (131.0, 161.5), turned to 45 degrees
- renumbered G*** to :3c
Routing:
- net /SCL: track 68.2 -> 331.2 mm
- net +3.3V: track 153.9 -> 367.0 mm
- net /GPIO3: track 46.8 -> 128.5 mm
- net /SDA: track 68.3 -> 147.0 mm
- net /GPI02: track 137.3 -> 208.4 mm
- net /DHT11 DATA: track 141.5 -> 194.4 mm
- net /ng: track 74.1 -> 108.0 mm
- net +5V: track 25.7 -> 59.0 mm
- net GND: track 438.6 -> 461.3 mm
- net /groundi: track 71.4 -> 88.7 mm
- net (no net): track 1.40 -> 0.00 mm

Commit message: changed
Parts:
- removed :3 (x4): LOGO, Imported Parts:abcd
- removed :3c (x2): LOGO, Imported Parts:def
- removed :3c: LOGO, LOGO
Other:
- board size 140 x 145.5 mm -> 114 x 128.5 mm
