File: Starbie/Starbie.kicad_sch (KiCad schematic)
At the start: 7 parts, among them J1 Conn_01x04_Pin, J2 Conn_01x08_Pin, SW1 SW_Push, SW2 SW_Push, U1 XIAO-ESP32-C3-SMD, U2 DHT11

Commit message: built schematic
Parts:
- J1: footprint (none) -> Imported Parts:Display_128x64_096_I2C
- J2: footprint (none) -> Connector_PinHeader_2.54mm:PinHeader_1x08_P2.54mm_Vertical
- R1: value R -> 10K; footprint Package_SO:TSOP-I-32_18.4x8mm_P0.5mm -> Resistor_THT:R_Axial_DIN0204_L3.6mm_D1.6mm_P7.62mm_Horizontal
- SW1: footprint Button_Switch_THT:SW_NKK_GW12LJP -> Button_Switch_Keyboard:SW_Cherry_MX_1.00u_PCB
- SW2: footprint (none) -> Button_Switch_Keyboard:SW_Cherry_MX_1.00u_PCB
- U1: footprint Seeed_Studio_XIAO_Series:XIAO-ESP32-C3-SMD -> Imported Parts:XIAO-ESP32-C6-DIP
Changed lines of the file:
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@@
 			)
 		)
-		(property "Footprint" ""
+		(property "Footprint" "Imported Parts:Display_128x64_096_I2C"
 			(at 38.1 105.41 0)
 			(hide yes)
@@
 			)
 		)
-		(property "Value" "R"
+		(property "Value" "10K"
 			(at 115.57 152.3999 0)
 			(show_name no)
@@
 			)
 		)
-		(property "Footprint" "Package_SO:TSOP-I-32_18.4x8mm_P0.5mm"
+		(property "Footprint" "Resistor_THT:R_Axial_DIN0204_L3.6mm_D1.6mm_P7.62mm_Horizontal"
 			(at 111.252 151.13 90)
 			(hide yes)
@@
 			)
 		)
-		(property "Footprint" "Button_Switch_THT:SW_NKK_GW12LJP"
+		(property "Footprint" "Button_Switch_Keyboard:SW_Cherry_MX_1.00u_PCB"
 			(at 41.91 68.58 0)
 			(hide yes)
@@
 			)
 		)
-		(property "Footprint" "Seeed_Studio_XIAO_Series:XIAO-ESP32-C3-SMD"
+		(property "Footprint" "Imported Parts:XIAO-ESP32-C6-DIP"
 			(at 51.562 113.284 0)
 			(hide yes)
@@
 			)
 		)
-		(property "Footprint" ""
+		(property "Footprint" "Connector_PinHeader_2.54mm:PinHeader_1x08_P2.54mm_Vertical"
 			(at 35.56 135.89 0)
 			(hide yes)
@@
 			)
 		)
-		(property "Footprint" ""
+		(property "Footprint" "Button_Switch_Keyboard:SW_Cherry_MX_1.00u_PCB"
 			(at 41.91 82.55 0)
 			(hide yes)

Commit message: changed
Parts:
- added J3: USB_C_Receptacle_USB2.0_14P, Connector_USB:USB_C_Receptacle_HRO_TYPE-C-31-M-17, symbol Connector:USB_C_Receptacle_USB2.0_14P
- added R2, R3: 5k, Package_DIP:DIP-8_W7.62mm, symbol Device:R
Connections:
- net +5V: now also J3.A4 (VBUS), J3.A9 (VBUS), J3.B4 (VBUS), J3.B9 (VBUS)
- net GND: now also J3.A1 (GND), J3.A12 (GND), J3.B1 (GND), J3.B12 (GND), J3.SH (SHIELD), R2.1, R3.1
- net pair2: now reaches U1.8 (D7)
- net pair2: now also J3.B7 (D-)
- net pair1: now reaches U1.9 (D8)
- net pair1: now also J3.A6 (D+), J3.A7 (D-), J3.B6 (D+)
- new net groundi: J3.B5 (CC2), R2.2
- new net ng: J3.A5 (CC1), R3.2
- no-connect marks 18 -> 16
